File: projects/step-motor-controller/step-motor-controller.kicad_sch (KiCad schematic)
At the start: 35 parts, among them J1 AC Input, J2 Motor, J3 Encoder, Q1 BC547, SW1 Limit-1, SW2 Limit-2, U1 OKI-78SR-5, U2 UART Display, U3 ESP32-DevKitC, U4 LV8729, U5 AM26LS32, U6 74HC4050

Commit message: feat: verified Step Motor Controller — 45-net schematic match, routed PCB, 0 electrical DRC, fab package
Parts:
- removed ?: (no value), symbol Connector_Generic:Conn_01x04
- removed C1: 100uF, Capacitor_THT:CP_Radial_D8.0mm_P3.50mm, symbol Device:CP
- removed C2: 10uF, Capacitor_THT:CP_Radial_D5.0mm_P2.50mm, symbol Device:CP
- removed R1, R3: FSR, Resistor_SMD:R_0805_2012Metric, symbol Device:R
- removed S1: Optic-1, OptoDevice:OptoDevice_TCRT5000, symbol Sensor_Optical:TCRT5000
- removed S2: Optic-2, OptoDevice:OptoDevice_TCRT5000, symbol Sensor_Optical:TCRT5000
- removed S3: Hall-1, Sensor:Sensor_Hall_TH, symbol Sensor_Magnetic:AH3503
- removed S4: Hall-2, Sensor:Sensor_Hall_TH, symbol Sensor_Magnetic:AH3503
- removed U1: OKI-78SR-5, Package_TO_SOT_THT:TO-220-3_Vertical, symbol Regulator_Switching:OKI-78SR-5_1.5-W36-C
- removed U3: ESP32-DevKitC, RF_Module:ESP32-DevKitC, symbol RF_Module:ESP32-DevKitC
- removed U4: LV8729, Package_SO:SOIC-16_3.9x9.9mm_P1.27mm, symbol Driver_Motor:LV8729
- removed U5: AM26LS32, Package_DIP:DIP-16_W7.62mm, symbol Interface:AM26LS32ACN
- removed U6: 74HC4050, Package_DIP:DIP-16_W7.62mm, symbol 74xx:74HC4050
- added C1: 100uF/35V, Capacitor_THT:CP_Radial_D6.3mm_P2.50mm, symbol Device:C_Polarized
- added C2: 10uF/16V, Capacitor_THT:CP_Radial_D5.0mm_P2.50mm, symbol Device:C_Polarized
- added R1, R3: FSR (external), Connector_PinHeader_2.54mm:PinHeader_1x02_P2.54mm_Vertical, symbol Connector_Generic:Conn_01x02
- added S1: Optic LS-1, Connector_PinHeader_2.54mm:PinHeader_1x03_P2.54mm_Vertical, symbol Connector_Generic:Conn_01x03
- added S2: Optic LS-2, Connector_PinHeader_2.54mm:PinHeader_1x03_P2.54mm_Vertical, symbol Connector_Generic:Conn_01x03
- added S3: Hall-1, Connector_PinHeader_2.54mm:PinHeader_1x03_P2.54mm_Vertical, symbol Connector_Generic:Conn_01x03
- added S4: Hall-2, Connector_PinHeader_2.54mm:PinHeader_1x03_P2.54mm_Vertical, symbol Connector_Generic:Conn_01x03
- added U1: OKI-78SR-5/1.5-W36-C, Converter_DCDC:Converter_DCDC_Murata_OKI-78SR_Vertical, symbol KicadAuto:OKI-78SR
- added U3: ESP32-DevKitC, AUTO:ESP32_SOCKET, symbol KicadAuto:ESP32-DevKitC
- added U4: LV8729 Module, AUTO:STEPSTICK_2x8, symbol KicadAuto:LV8729
- added U5: AM26LS32ACN, Package_DIP:DIP-16_W7.62mm, symbol KicadAuto:AM26LS32ACN
- added U6: 74HC4050N_652, Package_DIP:DIP-16_W7.62mm, symbol KicadAuto:74HC4050
- J1: value AC Input -> AC Input 3Pin; footprint Connector_PinHeader_2.54mm:PinHeader_1x03_P2.54mm_Vertical -> TerminalBlock_Phoenix:TerminalBlock_Phoenix_MKDS-1,5-3-5.08_1x03_P5.08mm_Horizontal
- J2: value Motor -> Step Motor; footprint Connector_PinHeader_2.54mm:PinHeader_1x04_P2.54mm_Vertical -> Connector_PinSocket_2.54mm:PinSocket_1x04_P2.54mm_Vertical
- J3: footprint Connector_PinHeader_2.54mm:PinHeader_1x08_P2.54mm_Vertical -> Connector_PinSocket_2.54mm:PinSocket_1x08_P2.54mm_Vertical
- PS1: footprint Converter_ACDC:ACDC-Converter_MeanWell_IRM-20 -> Converter_ACDC:Converter_ACDC_MeanWell_IRM-20-xx_THT
- SW1: value Limit-1 -> Limit SW-1; footprint Button_Switch_THT:SW_CuK_OS102011MA1QN1_SPDT_Angled -> Connector_PinHeader_2.54mm:PinHeader_1x03_P2.54mm_Vertical
- SW2: value Limit-2 -> Limit SW-2; footprint Button_Switch_THT:SW_CuK_OS102011MA1QN1_SPDT_Angled -> Connector_PinHeader_2.54mm:PinHeader_1x03_P2.54mm_Vertical
- U2: footprint Connector_PinHeader_2.54mm:PinHeader_1x04_P2.54mm_Vertical -> Connector_PinSocket_2.54mm:PinSocket_1x04_P2.54mm_Vertical
Connections:
- new net +24V: C1.1, PS1.4 (+Vo), U1.1 (VI), U4.16 (VM)
- new net +3V3: R1.1 (Pin_1), R11.1, R3.1 (Pin_1), R5.2, R6.2, U3.1 (3V3)
- new net +5V: C2.1, J3.1 (Pin_1), S1.1 (Pin_1), S2.1 (Pin_1), S3.1 (Pin_1), S4.1 (Pin_1), U1.3 (VO), U2.1 (Pin_1), U3.19 (5V), U4.10 (VDD), U5.16 (VCC), U5.4 (G), U6.1 (VCC)
- new net AC_L: J1.1 (Pin_1), PS1.1 (AC/L)
- new net AC_N: J1.2 (Pin_2), PS1.2 (AC/N)
- new net CHIP_PU: C5.1, Q1.1 (C), R11.2, U3.2 (EN)
- new net ENC_A_BUF: U5.3 (1Y), U6.3 (1A)
- new net ENC_A_N: J3.4 (Pin_4), U5.1 (1B)
- new net ENC_A_P: J3.3 (Pin_3), U5.2 (1A)
- new net ENC_B_BUF: U5.5 (2Y), U6.5 (2A)
- new net ENC_B_N: J3.6 (Pin_6), U5.6 (2A)
- new net ENC_B_P: J3.5 (Pin_5), U5.7 (2B)
- new net ENC_Z_BUF: U5.11 (3Y), U6.7 (3A)
- new net ENC_Z_ESP: U3.15 (GPIO13), U6.6 (3Y)
- new net ENC_Z_N: J3.8 (Pin_8), U5.10 (3A)
- new net ENC_Z_P: J3.7 (Pin_7), U5.9 (3B)
- new net FSR1_TOP: R1.2 (Pin_2), R2.1, U3.7 (GPIO32)
- new net FSR2_TOP: R3.2 (Pin_2), R4.1, U3.8 (GPIO33)
- new net GND: C1.2, C2.2, C3.2, C4.2, C5.2, J1.3 (Pin_3), J3.2 (Pin_2), PS1.3 (-Vo), Q1.3 (E), R10.1, R2.2, R4.2, R8.1, S1.3 (Pin_3), S2.3 (Pin_3), S3.2 (Pin_2), S4.2 (Pin_2), SW1.2 (B), SW2.2 (B), U1.2 (GND), U2.4 (Pin_4), U3.14 (GND), U4.15 (GND), U4.9 (GND), U5.12 (/G), U5.8 (GND), U6.8 (GND)
- new net GPIO18_OPTIC1: U3.30 (GPIO18), U6.10 (4Y)
- new net GPIO19_OPTIC2: U3.31 (GPIO19), U6.12 (5Y)
- new net GPIO21_ENC_A: U3.32 (GPIO21), U6.2 (1Y)
- new net GPIO22_ENC_B: U3.33 (GPIO22), U6.4 (2Y)
- new net GPIO23_RST: R12.1, U3.37 (GPIO23)
- new net HALL1_DIV: R7.2, R8.2, U3.5 (GPIO34)
- new net HALL1_RAW: R7.1, S3.3 (Pin_3)
- new net HALL2_DIV: R10.2, R9.2, U3.6 (GPIO35)
- new net HALL2_RAW: R9.1, S4.3 (Pin_3)
- new net MOT_1A: J2.1 (Pin_1), U4.14 (1A)
- new net MOT_1B: J2.2 (Pin_2), U4.13 (1B)
- new net MOT_2A: J2.3 (Pin_3), U4.12 (2A)
- new net MOT_2B: J2.4 (Pin_4), U4.11 (2B)
- new net M_DIR: U3.11 (GPIO27), U4.8 (DIR)
- new net M_EN: U3.12 (GPIO14), U4.1 (EN)
- new net M_MS1: U3.26 (GPIO4), U4.2 (MS1)
- new net M_MS2: U3.29 (GPIO5), U4.3 (MS2)
- new net M_MS3: U3.9 (GPIO25), U4.4 (MS3)
- new net M_STEP: U3.10 (GPIO26), U4.7 (STEP)
- new net OPTIC1_RAW: S1.2 (Pin_2), U6.9 (4A)
- new net OPTIC2_RAW: S2.2 (Pin_2), U6.11 (5A)
- new net Q1_BASE: Q1.2 (B), R12.2
- new net SW1_SIG: C3.1, R5.1, SW1.1 (A), U3.3 (GPIO36)
- new net SW2_SIG: C4.1, R6.1, SW2.1 (A), U3.4 (GPIO39)
- new net UART_M_RX: U2.3 (Pin_3), U3.28 (GPIO17)
- new net UART_M_TX: U2.2 (Pin_2), U3.27 (GPIO16)
Other:
- company: AutoGen -> (none)

Commit message: fix: no_connect markers on NC pins; PS1 Vo pins as power_out (ERC clean)
Connections:
- no-connect marks 0 -> 25
Changed lines of the file:
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@@
 		)
+	)
+	(no_connect
+		(at 217.2200 92.6200)
+	)
+	(no_connect
+		(at 217.2200 100.2400)
+	)
+	(no_connect
+		(at 217.2200 102.7800)
+	)
+	(no_connect
+		(at 217.2200 105.3200)
+	)
+	(no_connect
+		(at 252.7800 107.8600)
+	)
+	(no_connect
+		(at 252.7800 105.3200)
+	)
+	(no_connect
+		(at 252.7800 102.7800)
+	)
+	(no_connect
+		(at 252.7800 100.2400)
+	)
+	(no_connect
+		(at 252.7800 97.7000)
+	)
+	(no_connect
+		(at 252.7800 95.1600)
+	)
+	(no_connect
+		(at 252.7800 72.3000)
+	)
+	(no_connect
+		(at 252.7800 69.7600)
+	)
+	(no_connect
+		(at 252.7800 67.2200)
+	)
+	(no_connect
+		(at 252.7800 62.1400)
+	)
+	(no_connect
+		(at 302.3000 86.2700)
+	)
+	(no_connect
+		(at 302.3000 88.8100)
+	)
+	(no_connect
+		(at 87.7000 113.7300)
+	)
+	(no_connect
+		(at 87.7000 111.1900)
+	)
+	(no_connect
+		(at 87.7000 108.6500)
+	)
+	(no_connect
+		(at 147.7000 113.7300)
+	)
+	(no_connect
+		(at 147.7000 111.1900)
+	)
+	(no_connect
+		(at 147.7000 108.6500)
+	)
+	(no_connect
+		(at 147.7000 106.1100)
+	)
+	(no_connect
+		(at 40.0800 167.5400)
+	)
+	(no_connect
+		(at 40.0800 189.5400)
 	)
 	(global_label
