File: projects/step-motor-controller/step-motor-controller.kicad_sch (KiCad schematic)
At the start: 34 parts, among them J1 AC Input 3Pin, J2 Step Motor, J3 Encoder, Q1 BC547, SW1 Limit SW-1, SW2 Limit SW-2, U1 OKI-78SR-5/1.5-W36-C, U2 UART Display, U3 ESP32-DevKitC, U4 LV8729 Module, U5 AM26LS32ACN, U6 74HC4050N_652

Commit message: feat: wired schematic v4 - 45/45 nets match Excel, 0 ERC, rails+wires+labels
Parts:
- C1: footprint Capacitor_THT:CP_Radial_D6.3mm_P2.50mm -> (none)
- C2: footprint Capacitor_THT:CP_Radial_D5.0mm_P2.50mm -> (none)
- C3, C4, C5: footprint Capacitor_SMD:C_0805_2012Metric -> (none)
- J1: value AC Input 3Pin -> AC Input
- R10, R11, R12, R2, R4, R5, R6, R7, R8, R9: footprint Resistor_SMD:R_0805_2012Metric -> (none)
- SW1: value Limit SW-1 -> SW1
- SW2: value Limit SW-2 -> SW2
- U1: value OKI-78SR-5/1.5-W36-C -> OKI-78SR-5
- U6: value 74HC4050N_652 -> 74HC4050N
