File: projects/step-motor-controller/schematic-package/step-motor-controller.kicad_sch (KiCad schematic)
At the start: 34 parts, among them J1 AC Input, J2 Step Motor, J3 Encoder, Q1 BC547, SW1 SW1, SW2 SW2, U1 OKI-78SR-5, U2 UART Display, U3 ESP32-DevKitC, U4 LV8729 Module, U5 AM26LS32ACN, U6 74HC4050N

Commit message: feat: THT conversion - all passives through-hole (DIN0207 resistors, film/electrolytic caps), 45/45 nets, 0 ERC
Parts:
- C1: footprint (none) -> Capacitor_THT:CP_Radial_D8.0mm_P3.50mm
- C2: footprint (none) -> Capacitor_THT:CP_Radial_D6.3mm_P2.50mm
- C3, C4, C5: footprint (none) -> Capacitor_THT:C_Rect_L7.0mm_W2.5mm_P5.00mm
- R10, R11, R12, R2, R4, R5, R6, R7, R8, R9: footprint (none) -> Resistor_THT:R_Axial_DIN0207_L6.3mm_D2.5mm_P10.16mm_Horizontal
Changed lines of the file:
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@@
 		(property "Reference" "C1" (at 204.47 66.85 0) (effects (font (size 1.27 1.27))))
 		(property "Value" "100uF/35V" (at 204.47 72.85 0) (effects (font (size 1.27 1.27))))
-		(property "Footprint" "" (at 204.47 69.85 0) (effects (font (size 1.27 1.27)) hide))
+		(property "Footprint" "Capacitor_THT:CP_Radial_D8.0mm_P3.50mm" (at 204.47 69.85 0) (effects (font (size 1.27 1.27)) hide))
 		(property "Datasheet" "" (at 204.47 69.85 0) (effects (font (size 1.27 1.27)) hide))
 		(property "Description" "100uF/35V" (at 204.47 69.85 0) (effects (font (size 1.27 1.27)) hide))
@@
 		(property "Reference" "C2" (at 222.25 66.85 0) (effects (font (size 1.27 1.27))))
 		(property "Value" "10uF/16V" (at 222.25 72.85 0) (effects (font (size 1.27 1.27))))
-		(property "Footprint" "" (at 222.25 69.85 0) (effects (font (size 1.27 1.27)) hide))
+		(property "Footprint" "Capacitor_THT:CP_Radial_D6.3mm_P2.50mm" (at 222.25 69.85 0) (effects (font (size 1.27 1.27)) hide))
 		(property "Datasheet" "" (at 222.25 69.85 0) (effects (font (size 1.27 1.27)) hide))
 		(property "Description" "10uF/16V" (at 222.25 69.85 0) (effects (font (size 1.27 1.27)) hide))
@@
 		(property "Reference" "R11" (at 204.47 121.46 0) (effects (font (size 1.27 1.27))))
 		(property "Value" "10K" (at 204.47 127.46 0) (effects (font (size 1.27 1.27))))
-		(property "Footprint" "" (at 204.47 124.46 0) (effects (font (size 1.27 1.27)) hide))
+		(property "Footprint" "Resistor_THT:R_Axial_DIN0207_L6.3mm_D2.5mm_P10.16mm_Horizontal" (at 204.47 124.46 0) (effects (font (size 1.27 1.27)) hide))
 		(property "Datasheet" "" (at 204.47 124.46 0) (effects (font (size 1.27 1.27)) hide))
 		(property "Description" "10K" (at 204.47 124.46 0) (effects (font (size 1.27 1.27)) hide))
@@
 		(property "Reference" "C5" (at 218.44 139.24 0) (effects (font (size 1.27 1.27))))
 		(property "Value" "100nF" (at 218.44 145.24 0) (effects (font (size 1.27 1.27))))
-		(property "Footprint" "" (at 218.44 142.24 0) (effects (font (size 1.27 1.27)) hide))
+		(property "Footprint" "Capacitor_THT:C_Rect_L7.0mm_W2.5mm_P5.00mm" (at 218.44 142.24 0) (effects (font (size 1.27 1.27)) hide))
 		(property "Datasheet" "" (at 218.44 142.24 0) (effects (font (size 1.27 1.27)) hide))
 		(property "Description" "100nF" (at 218.44 142.24 0) (effects (font (size 1.27 1.27)) hide))
@@
 		(property "Reference" "R12" (at 294.64 115.11 0) (effects (font (size 1.27 1.27))))
 		(property "Value" "1K" (at 294.64 121.11 0) (effects (font (size 1.27 1.27))))
-		(property "Footprint" "" (at 294.64 118.11 0) (effects (font (size 1.27 1.27)) hide))
+		(property "Footprint" "Resistor_THT:R_Axial_DIN0207_L6.3mm_D2.5mm_P10.16mm_Horizontal" (at 294.64 118.11 0) (effects (font (size 1.27 1.27)) hide))
 		(property "Datasheet" "" (at 294.64 118.11 0) (effects (font (size 1.27 1.27)) hide))
 		(property "Description" "1K" (at 294.64 118.11 0) (effects (font (size 1.27 1.27)) hide))
@@
 		(property "Reference" "R5" (at 165.1 118.92 0) (effects (font (size 1.27 1.27))))
 		(property "Value" "10K" (at 165.1 124.92 0) (effects (font (size 1.27 1.27))))
-		(property "Footprint" "" (at 165.1 121.92 0) (effects (font (size 1.27 1.27)) hide))
+		(property "Footprint" "Resistor_THT:R_Axial_DIN0207_L6.3mm_D2.5mm_P10.16mm_Horizontal" (at 165.1 121.92 0) (effects (font (size 1.27 1.27)) hide))
 		(property "Datasheet" "" (at 165.1 121.92 0) (effects (font (size 1.27 1.27)) hide))
 		(property "Description" "10K" (at 165.1 121.92 0) (effects (font (size 1.27 1.27)) hide))
@@
 		(property "Reference" "R6" (at 165.1 136.7 0) (effects (font (size 1.27 1.27))))
 		(property "Value" "10K" (at 165.1 142.7 0) (effects (font (size 1.27 1.27))))
-		(property "Footprint" "" (at 165.1 139.7 0) (effects (font (size 1.27 1.27)) hide))
+		(property "Footprint" "Resistor_THT:R_Axial_DIN0207_L6.3mm_D2.5mm_P10.16mm_Horizontal" (at 165.1 139.7 0) (effects (font (size 1.27 1.27)) hide))
 		(property "Datasheet" "" (at 165.1 139.7 0) (effects (font (size 1.27 1.27)) hide))
 		(property "Description" "10K" (at 165.1 139.7 0) (effects (font (size 1.27 1.27)) hide))
@@
 		(property "Reference" "C3" (at 187.96 118.92 0) (effects (font (size 1.27 1.27))))
 		(property "Value" "100nF" (at 187.96 124.92 0) (effects (font (size 1.27 1.27))))
-		(property "Footprint" "" (at 187.96 121.92 0) (effects (font (size 1.27 1.27)) hide))
+		(property "Footprint" "Capacitor_THT:C_Rect_L7.0mm_W2.5mm_P5.00mm" (at 187.96 121.92 0) (effects (font (size 1.27 1.27)) hide))
 		(property "Datasheet" "" (at 187.96 121.92 0) (effects (font (size 1.27 1.27)) hide))
 		(property "Description" "100nF" (at 187.96 121.92 0) (effects (font (size 1.27 1.27)) hide))
@@
 		(property "Reference" "C4" (at 187.96 136.7 0) (effects (font (size 1.27 1.27))))
 		(property "Value" "100nF" (at 187.96 142.7 0) (effects (font (size 1.27 1.27))))
-		(property "Footprint" "" (at 187.96 139.7 0) (effects (font (size 1.27 1.27)) hide))
+		(property "Footprint" "Capacitor_THT:C_Rect_L7.0mm_W2.5mm_P5.00mm" (at 187.96 139.7 0) (effects (font (size 1.27 1.27)) hide))
 		(property "Datasheet" "" (at 187.96 139.7 0) (effects (font (size 1.27 1.27)) hide))
 		(property "Description" "100nF" (at 187.96 139.7 0) (effects (font (size 1.27 1.27)) hide))
@@
 		(property "Reference" "R7" (at 100.33 196.39 0) (effects (font (size 1.27 1.27))))
 		(property "Value" "10K" (at 100.33 202.39 0) (effects (font (size 1.27 1.27))))
-		(property "Footprint" "" (at 100.33 199.39 0) (effects (font (size 1.27 1.27)) hide))
+		(property "Footprint" "Resistor_THT:R_Axial_DIN0207_L6.3mm_D2.5mm_P10.16mm_Horizontal" (at 100.33 199.39 0) (effects (font (size 1.27 1.27)) hide))
 		(property "Datasheet" "" (at 100.33 199.39 0) (effects (font (size 1.27 1.27)) hide))
 		(property "Description" "10K" (at 100.33 199.39 0) (effects (font (size 1.27 1.27)) hide))
@@
 		(property "Reference" "R8" (at 111.76 196.39 0) (effects (font (size 1.27 1.27))))
 		(property "Value" "20K" (at 111.76 202.39 0) (effects (font (size 1.27 1.27))))
-		(property "Footprint" "" (at 111.76 199.39 0) (effects (font (size 1.27 1.27)) hide))
+		(property "Footprint" "Resistor_THT:R_Axial_DIN0207_L6.3mm_D2.5mm_P10.16mm_Horizontal" (at 111.76 199.39 0) (effects (font (size 1.27 1.27)) hide))
 		(property "Datasheet" "" (at 111.76 199.39 0) (effects (font (size 1.27 1.27)) hide))
 		(property "Description" "20K" (at 111.76 199.39 0) (effects (font (size 1.27 1.27)) hide))
@@
 		(property "Reference" "R9" (at 134.62 196.39 0) (effects (font (size 1.27 1.27))))
 		(property "Value" "10K" (at 134.62 202.39 0) (effects (font (size 1.27 1.27))))
-		(property "Footprint" "" (at 134.62 199.39 0) (effects (font (size 1.27 1.27)) hide))
+		(property "Footprint" "Resistor_THT:R_Axial_DIN0207_L6.3mm_D2.5mm_P10.16mm_Horizontal" (at 134.62 199.39 0) (effects (font (size 1.27 1.27)) hide))
 		(property "Datasheet" "" (at 134.62 199.39 0) (effects (font (size 1.27 1.27)) hide))
 		(property "Description" "10K" (at 134.62 199.39 0) (effects (font (size 1.27 1.27)) hide))
@@
 		(property "Reference" "R10" (at 147.32 196.39 0) (effects (font (size 1.27 1.27))))
 		(property "Value" "20K" (at 147.32 202.39 0) (effects (font (size 1.27 1.27))))
-		(property "Footprint" "" (at 147.32 199.39 0) (effects (font (size 1.27 1.27)) hide))
+		(property "Footprint" "Resistor_THT:R_Axial_DIN0207_L6.3mm_D2.5mm_P10.16mm_Horizontal" (at 147.32 199.39 0) (effects (font (size 1.27 1.27)) hide))
 		(property "Datasheet" "" (at 147.32 199.39 0) (effects (font (size 1.27 1.27)) hide))
 		(property "Description" "20K" (at 147.32 199.39 0) (effects (font (size 1.27 1.27)) hide))
@@
 		(property "Reference" "R2" (at 115.57 233.22 0) (effects (font (size 1.27 1.27))))
 		(property "Value" "10K" (at 115.57 239.22 0) (effects (font (size 1.27 1.27))))
-		(property "Footprint" "" (at 115.57 236.22 0) (effects (font (size 1.27 1.27)) hide))
+		(property "Footprint" "Resistor_THT:R_Axial_DIN0207_L6.3mm_D2.5mm_P10.16mm_Horizontal" (at 115.57 236.22 0) (effects (font (size 1.27 1.27)) hide))
 		(property "Datasheet" "" (at 115.57 236.22 0) (effects (font (size 1.27 1.27)) hide))
 		(property "Description" "10K" (at 115.57 236.22 0) (effects (font (size 1.27 1.27)) hide))
@@
 		(property "Reference" "R4" (at 154.94 233.22 0) (effects (font (size 1.27 1.27))))
 		(property "Value" "10K" (at 154.94 239.22 0) (effects (font (size 1.27 1.27))))
-		(property "Footprint" "" (at 154.94 236.22 0) (effects (font (size 1.27 1.27)) hide))
+		(property "Footprint" "Resistor_THT:R_Axial_DIN0207_L6.3mm_D2.5mm_P10.16mm_Horizontal" (at 154.94 236.22 0) (effects (font (size 1.27 1.27)) hide))
 		(property "Datasheet" "" (at 154.94 236.22 0) (effects (font (size 1.27 1.27)) hide))
 		(property "Description" "10K" (at 154.94 236.22 0) (effects (font (size 1.27 1.27)) hide))
